Commit message: [update]完成仿真包的ros jazzy迁移

File: src/rm_27_stimulation/urdf/mid360.xacro (robot description, xacro)
@@ -34,42 +34,37 @@
     </joint>
     <gazebo reference="${name}">
-      <sensor type="ray" name="${name}">
+      <sensor type="gpu_lidar" name="${name}">
         <pose>0 0 0 0 0 0</pose>
         <always_on>true</always_on>
-        <visualize>true</visualize>
+        <visualize>false</visualize>
         <update_rate>10</update_rate>
-        <plugin name="${name}_plugin" filename="libros2_livox.so">
-          <ray>
-            <scan>
-              <horizontal>
-                <samples>100</samples>
-                <resolution>1</resolution>
-                <min_angle>${0}</min_angle>
-                <max_angle>${2*M_PI}</max_angle>
-              </horizontal>
-              <vertical>
-                <samples>360</samples>
-                <resolution>1</resolution>
-                <min_angle>${-7.22/180*M_PI}</min_angle>
-                <max_angle>${55.22/180*M_PI}</max_angle>
-              </vertical>
-            </scan>
-            <range>
-              <min>${laser_min_range}</min>
-              <max>${laser_max_range}</max>
-              <resolution>${resolution}</resolution>
-            </range>
-            <noise>
-              <type>gaussian</type>
-              <mean>${noise_mean}</mean>
-              <stddev>${noise_stddev}</stddev>
-            </noise>
-          </ray>
-          <visualize>false</visualize>
-          <samples>${samples}</samples>
-          <downsample>1</downsample>
-          <csv_file_name>$(find rm_27_stimulation)/scan_mode/mid360.csv</csv_file_name>
-          <topic>${topic}</topic>
-        </plugin>
+        <topic>${topic}</topic>
+        <gz_frame_id>${name}</gz_frame_id>
+        <lidar>
+          <scan>
+            <horizontal>
+              <samples>100</samples>
+              <resolution>1</resolution>
+              <min_angle>${0}</min_angle>
+              <max_angle>${2*M_PI}</max_angle>
+            </horizontal>
+            <vertical>
+              <samples>360</samples>
+              <resolution>1</resolution>
+              <min_angle>${-7.22/180*M_PI}</min_angle>
+              <max_angle>${55.22/180*M_PI}</max_angle>
+            </vertical>
+          </scan>
+          <range>
+            <min>${laser_min_range}</min>
+            <max>${laser_max_range}</max>
+            <resolution>${resolution}</resolution>
+          </range>
+          <noise>
+            <type>gaussian</type>
+            <mean>${noise_mean}</mean>
+            <stddev>${noise_stddev}</stddev>
+          </noise>
+        </lidar>
       </sensor>
     </gazebo>

File: src/rm_27_stimulation/urdf/simulation_waking_robot.xacro (robot description, xacro)
@@ -114,27 +114,21 @@
     <xacro:default_inertial mass="0.5"/>
   </link>
-  <joint name="base_to_wheel1" type="continuous">
+  <joint name="base_to_wheel1" type="fixed">
     <parent link="base_link"/>
     <child link="wheel_1"/>
     <origin rpy="${-PI/2} 0 0" xyz="0.1 0.13 0"/>
-    <axis xyz="0 0 1" />
-  </joint>
-  <joint name="base_to_wheel2" type="continuous">
-    <axis xyz="0 0 1" />
-    <anchor xyz="0 0 0" />
-    <limit effort="100" velocity="100" />
+  </joint>
+  <joint name="base_to_wheel2" type="fixed">
     <parent link="base_link"/>
     <child link="wheel_2"/>
     <origin rpy="${-PI/2} 0 0" xyz="-0.1 0.13 0"/>
   </joint>
-  <joint name="base_to_wheel3" type="continuous">
-    <parent link="base_link"/>
-    <axis xyz="0 0 1" />
+  <joint name="base_to_wheel3" type="fixed">
+    <parent link="base_link"/>
     <child link="wheel_3"/>
     <origin rpy="${-PI/2} 0 0" xyz="0.1 -0.13 0"/>
   </joint>
-  <joint name="base_to_wheel4" type="continuous">
-    <parent link="base_link"/>
-    <axis xyz="0 0 1" />
+  <joint name="base_to_wheel4" type="fixed">
+    <parent link="base_link"/>
     <child link="wheel_4"/>
     <origin rpy="${-PI/2} 0 0" xyz="-0.1 -0.13 0"/>
@@ -192,44 +186,21 @@
     <material>Gazebo/LightBlueLaser</material>
   </gazebo>
-  <!-- Drive controller plugin-->
-  <!-- https://github.com/ros-simulation/gazebo_ros_pkgs/wiki/ROS-2-Migration:-Planar-Move -->
+  <!-- Drive controller plugin -->
   <gazebo>
-    <plugin name="mecanum_controller" filename="libgazebo_ros_planar_move.so">
-      <ros>
-        <!-- Add a namespace -->
-        <namespace>/</namespace>
-        <!-- Remap the default topic -->
-        <remapping>cmd_vel:=cmd_vel</remapping>
-        <remapping>odom:=gazebo_odom_unused</remapping>
-      </ros>
-      <!-- Set control loop update rate -->
-      <update_rate>100</update_rate>
-      <!-- Set odom publish rate -->
-      <publish_rate>10</publish_rate>
-      <!-- Set if odom required -->
-      <publish_odom>false</publish_odom>
-      <publish_odom_tf>false</publish_odom_tf>
-      <!-- Frame IDs -->
-      <odometry_frame>gazebo_odom_unused</odometry_frame>
-      <robot_base_frame>gazebo_base_footprint_unused</robot_base_frame>
-      <!-- Set odom covariance -->
-      <covariance_x>0.0001</covariance_x>
-      <covariance_y>0.0001</covariance_y>
-      <covariance_yaw>0.01</covariance_yaw>
+    <plugin name="rm_27_stimulation::CmdVelPoseControlSystem" filename="librm27_cmd_vel_pose_control_system.so">
+      <topic>/cmd_vel</topic>
+      <body_frame>true</body_frame>
+      <command_timeout>0.5</command_timeout>
+      <max_linear_velocity>3.0</max_linear_velocity>
+      <max_angular_velocity>6.0</max_angular_velocity>
     </plugin>
   </gazebo>
   <!-- mid360_imu plugin -->
-  <!-- https://github.com/ros-simulation/gazebo_ros_pkgs/wiki/ROS-2-Migration:-IMU-Sensors -->
   <gazebo reference="imu_link">
     <sensor name="mid360_imu" type="imu">
       <always_on>true</always_on>
       <update_rate>100</update_rate>
-      <plugin name="imu_plugin" filename="libgazebo_ros_imu_sensor.so">
-        <ros>
-          <namespace>/</namespace>
-          <remapping>~/out:=/livox/imu</remapping>
-        </ros>
-        <frame_name>imu_link</frame_name>
-      </plugin>
+      <topic>/livox/imu</topic>
+      <gz_frame_id>imu_link</gz_frame_id>
     </sensor>
   </gazebo>

Commit message: [update]添加ROGMap三维空间感知与minco规划期与mpc控制器

File: src/rm_27_stimulation/urdf/mid360.xacro (robot description, xacro)
@@ -44,5 +44,7 @@
           <scan>
             <horizontal>
-              <samples>100</samples>
+              <!-- Keep azimuth spacing below one 5 cm ROG cell at the
+                   near-ground return radius. -->
+              <samples>360</samples>
               <resolution>1</resolution>
               <min_angle>${0}</min_angle>
@@ -50,5 +52,8 @@
             </horizontal>
             <vertical>
-              <samples>360</samples>
+              <!-- 320 elevation rings keep the nearest ground-return spacing
+                   below one 5 cm ROG cell while bounding Gazebo, DDS, and map
+                   update load; total rays are 115200. -->
+              <samples>320</samples>
               <resolution>1</resolution>
               <min_angle>${-7.22/180*M_PI}</min_angle>

File: src/rm_27_stimulation/urdf/simulation_waking_robot.xacro (robot description, xacro)
@@ -3,4 +3,7 @@
   <xacro:property name="length_wheel" value="0.05" />
   <xacro:property name="radius_wheel" value="0.06" />
+  <xacro:property name="omni_contact_radius" value="${radius_wheel}" />
+  <xacro:property name="omni_contact_x_inset" value="0.02" />
+  <xacro:property name="omni_contact_y_inset" value="0.04" />
   <xacro:property name="PI" value="3.1415926"/>
   <xacro:macro name="default_inertial" params="mass">
@@ -55,6 +58,11 @@
     </visual>
     <collision>
-      <geometry>
-        <cylinder length="${length_wheel}" radius="${radius_wheel}"/>
+      <!-- The real chassis is holonomic. Full wheel-radius spherical contacts
+           preserve curb/ramp traversal without imposing a fixed cylinder axle
+           direction on DART. The centers are inset so their 0.28 x 0.30 m
+           envelope remains inside the configured 0.32 x 0.31 m footprint. -->
+      <origin xyz="${-omni_contact_x_inset} 0 ${-omni_contact_y_inset}" rpy="0 0 0"/>
+      <geometry>
+        <sphere radius="${omni_contact_radius}"/>
       </geometry>
     </collision>
@@ -70,6 +78,7 @@
     </visual>
     <collision>
-      <geometry>
-        <cylinder length="${length_wheel}" radius="${radius_wheel}"/>
+      <origin xyz="${omni_contact_x_inset} 0 ${-omni_contact_y_inset}" rpy="0 0 0"/>
+      <geometry>
+        <sphere radius="${omni_contact_radius}"/>
       </geometry>
     </collision>
@@ -85,6 +94,7 @@
     </visual>
     <collision>
-      <geometry>
-        <cylinder length="${length_wheel}" radius="${radius_wheel}"/>
+      <origin xyz="${-omni_contact_x_inset} 0 ${omni_contact_y_inset}" rpy="0 0 0"/>
+      <geometry>
+        <sphere radius="${omni_contact_radius}"/>
       </geometry>
     </collision>
@@ -100,6 +110,7 @@
     </visual>
     <collision>
-      <geometry>
-        <cylinder length="${length_wheel}" radius="${radius_wheel}"/>
+      <origin xyz="${omni_contact_x_inset} 0 ${omni_contact_y_inset}" rpy="0 0 0"/>
+      <geometry>
+        <sphere radius="${omni_contact_radius}"/>
       </geometry>
     </collision>
@@ -195,6 +206,17 @@
       <max_angular_velocity>6.0</max_angular_velocity>
       <linear_velocity_gain>80.0</linear_velocity_gain>
+      <!-- The 11.8-degree, low-friction test ramp needs about 21 N to hold this 10.2 kg model. -->
+      <linear_velocity_integral_gain>45.0</linear_velocity_integral_gain>
       <angular_velocity_gain>4.0</angular_velocity_gain>
       <max_planar_force>120.0</max_planar_force>
+      <max_planar_integral_force>35.0</max_planar_integral_force>
+      <!-- Add force only after measured motion stalls along a non-zero command.
+           It clears at 0.10 m/s, so no breakaway impulse remains on the slope. -->
+      <stall_assist_command_threshold>0.08</stall_assist_command_threshold>
+      <stall_assist_engage_velocity>0.02</stall_assist_engage_velocity>
+      <stall_assist_release_velocity>0.10</stall_assist_release_velocity>
+      <stall_assist_delay>0.20</stall_assist_delay>
+      <stall_assist_ramp_rate>100.0</stall_assist_ramp_rate>
+      <max_stall_assist_force>45.0</max_stall_assist_force>
       <max_yaw_torque>8.0</max_yaw_torque>
     </plugin>

File: src/sentry_robot_description/urdf/sentry_robot.urdf.xacro (robot description, xacro)
@@ -3,5 +3,5 @@
   <xacro:arg name="base_to_gimbal_xyz" default="0 0 0.12"/>
   <xacro:arg name="base_to_gimbal_rpy" default="0 0 0"/>
-  <xacro:arg name="base_to_lidar_xyz" default="0.0 0.18 0.28"/>
+  <xacro:arg name="base_to_lidar_xyz" default="0.0 -0.18 0.28"/>
   <xacro:arg name="base_to_lidar_rpy" default="0 0 0"/>
   <xacro:arg name="base_to_imu_xyz" default="$(arg base_to_lidar_xyz)"/>
