Commit message: [update]引入仿真世界场地碰撞模型；用solidwork导入仿真小车模型，同时更改一版适用的仿真参数；启动gazebo或者rviz时使用核显加速

File: src/rm_27_stimulation/urdf/mid360.xacro (robot description, xacro)
@@ -9,7 +9,7 @@
   <xacro:property name="noise_stddev" value="0.002"/>
   <xacro:property name="mass" value="0.4" />
-  <xacro:property name="length" value="0.1" />
-  <xacro:property name="width" value="0.06" />
-  <xacro:property name="height" value="0.06" />
+  <xacro:property name="length" value="0.076" />
+  <xacro:property name="width" value="0.072" />
+  <xacro:property name="height" value="0.066" />
   <xacro:macro name="box_inertia" params="m w h d">
     <inertial>
@@ -19,12 +19,13 @@
     </inertial>
   </xacro:macro>
-  <xacro:macro name="mid360" params="name:='' parent:= 'base_link' topic:='mid360' noise_mean:='0.0' noise_stddev:='0.002' *origin ">
+  <xacro:macro name="mid360" params="name:='' parent:= 'base_link' topic:='mid360' noise_mean:='0.0' noise_stddev:='0.002' hide_visual:='false' *origin ">
     <link name="${name}">
-      <visual>
-        <origin xyz="0.025 -0.0265 -0.025" rpy="${pi/2} 0 ${pi}"/>
-        <geometry>
-          <box size="${length} ${width} ${height}"/>
-        </geometry>
-      </visual>
+      <xacro:unless value="${hide_visual}">
+        <visual>
+          <geometry>
+            <box size="${length} ${width} ${height}"/>
+          </geometry>
+        </visual>
+      </xacro:unless>
     </link>
     <joint name="${name}_joint" type="fixed">

File: src/rm_27_stimulation/urdf/simulation_waking_robot.xacro (robot description, xacro)
@@ -1,37 +1,98 @@
 <?xml version="1.0"?>
 <robot name="robot" xmlns:xacro="http://www.ros.org/wiki/xacro">
-  <xacro:property name="length_wheel" value="0.05" />
-  <xacro:property name="radius_wheel" value="0.06" />
+  <xacro:arg name="use_cad_visual" default="true" />
+  <xacro:arg name="cad_visual_scale" default="1.0" />
+  <xacro:property name="length_wheel" value="0.065" />
+  <xacro:property name="radius_wheel" value="0.080" />
   <xacro:property name="omni_contact_radius" value="${radius_wheel}" />
-  <xacro:property name="omni_contact_x_inset" value="0.02" />
-  <xacro:property name="omni_contact_y_inset" value="0.04" />
+  <xacro:property name="wheel_center_offset" value="0.218" />
+  <xacro:property name="omni_friction" value="0.05" />
+  <xacro:property name="body_mass" value="8.2" />
+  <xacro:property name="wheel_mass" value="0.5" />
   <xacro:property name="PI" value="3.1415926"/>
-  <xacro:macro name="default_inertial" params="mass">
+  <material name="cad_body"><color rgba="0.26 0.29 0.32 1" /></material>
+  <material name="cad_wheels"><color rgba="0.025 0.025 0.028 1" /></material>
+  <material name="cad_armor"><color rgba="0.62 0.035 0.035 1" /></material>
+  <material name="cad_sensors"><color rgba="0.08 0.24 0.30 1" /></material>
+  <xacro:macro name="box_inertial" params="mass x y z ox oy oz">
+    <inertial>
+      <origin xyz="${ox} ${oy} ${oz}" rpy="0 0 0" />
+      <mass value="${mass}" />
+      <inertia ixx="${mass * (y*y + z*z) / 12.0}" ixy="0.0" ixz="0.0"
+               iyy="${mass * (x*x + z*z) / 12.0}" iyz="0.0"
+               izz="${mass * (x*x + y*y) / 12.0}" />
+    </inertial>
+  </xacro:macro>
+  <xacro:macro name="sphere_inertial" params="mass radius">
     <inertial>
       <mass value="${mass}" />
-      <inertia ixx="0.01" ixy="0.0" ixz="0.0"
-                    iyy="0.01" iyz="0.0" izz="0.01" />
+      <inertia ixx="${0.4 * mass * radius * radius}" ixy="0.0" ixz="0.0"
+               iyy="${0.4 * mass * radius * radius}" iyz="0.0"
+               izz="${0.4 * mass * radius * radius}" />
     </inertial>
   </xacro:macro>
-  <!-- Logical Mid360 frame relative to base_link; physical roll is compensated before this frame. -->
-  <xacro:arg name="xyz" default="0.0 0.18 0.14" />
-  <xacro:arg name="rpy" default="0 0 0" />
+  <xacro:macro name="cad_visual" params="mesh material">
+    <visual>
+      <geometry>
+        <mesh filename="package://rm_27_stimulation/meshes/rm27_sentry_visual/${mesh}.stl"
+              scale="$(arg cad_visual_scale) $(arg cad_visual_scale) $(arg cad_visual_scale)" />
+      </geometry>
+      <material name="${material}" />
+    </visual>
+  </xacro:macro>
+  <!-- mu1/mu2 are converted only to ODE friction. Keep Bullet explicit so
+       changing physics engines does not silently restore its default 1.0. -->
+  <xacro:macro name="bullet_omni_friction">
+    <collision>
+      <surface>
+        <friction>
+          <bullet>
+            <friction>${omni_friction}</friction>
+            <friction2>${omni_friction}</friction2>
+            <rolling_friction>0.0</rolling_friction>
+          </bullet>
+        </friction>
+      </surface>
+    </collision>
+  </xacro:macro>
+  <!-- CAD gimbals face +X; keep the original +Y mount with -30 deg roll. -->
+  <xacro:arg name="xyz" default="0.0 0.126 0.130" />
+  <xacro:arg name="rpy" default="-0.523598775598 0 0" />
   <link name="base_link">
-    <visual>
-      <geometry>
-        <box size="0.2 .3 .14"/>
-      </geometry>
-      <origin rpy="0 0 ${PI/2}" xyz="0 0 0.07"/>
-      <material name="orange">
-        <color rgba="0.95 0.28 0.04 1"/>
-      </material>
-    </visual>
-    <collision>
-      <geometry>
-        <box size="0.2 .3 0.14"/>
-      </geometry>
-      <origin rpy="0 0 ${PI/2}" xyz="0 0 0.07"/>
-    </collision>
-    <xacro:default_inertial mass="8.2"/>
+    <xacro:if value="$(arg use_cad_visual)">
+      <xacro:cad_visual mesh="body" material="cad_body" />
+      <xacro:cad_visual mesh="wheels" material="cad_wheels" />
+      <xacro:cad_visual mesh="armor" material="cad_armor" />
+      <xacro:cad_visual mesh="sensors" material="cad_sensors" />
+    </xacro:if>
+    <xacro:unless value="$(arg use_cad_visual)">
+      <visual>
+        <geometry>
+          <cylinder radius="0.375" length="0.12" />
+        </geometry>
+        <origin rpy="0 0 0" xyz="0 0 0.06" />
+        <material name="orange">
+          <color rgba="0.95 0.28 0.04 1" />
+        </material>
+      </visual>
+    </xacro:unless>
+    <!-- The new wire-free CAD is a 0.592 x 0.594 m rounded-square chassis.
+         Four wheel spheres below model its diagonal corners. -->
+    <collision>
+      <geometry>
+        <cylinder radius="0.280" length="0.12" />
+      </geometry>
+      <origin rpy="0 0 0" xyz="0 0 0.06" />
+    </collision>
+    <collision>
+      <geometry>
+        <box size="0.48 0.48 0.08" />
+      </geometry>
+      <origin rpy="0 0 0" xyz="0 0 0.14" />
+    </collision>
+    <!-- STL has no material density. Preserve the validated 10.2 kg total
+         mass, but derive the inertia from the CAD body envelope. -->
+    <xacro:box_inertial mass="${body_mass}" x="0.54" y="0.54" z="0.20"
+                         ox="0.0" oy="0.0" oz="0.066" />
   </link>
   <link name="base_footprint"/>
@@ -48,92 +109,71 @@
   </joint>
   <link name="wheel_1">
-    <visual>
-      <geometry>
-        <cylinder length="${length_wheel}" radius="${radius_wheel}"/>
-      </geometry>
-      <origin rpy="0 0 0" xyz="0 0 0"/>
-      <material name="black">
-        <color rgba="0 0 0 1"/>
-      </material>
-    </visual>
-    <collision>
-      <!-- The real chassis is holonomic. Full wheel-radius spherical contacts
-           preserve curb/ramp traversal without imposing a fixed cylinder axle
-           direction on DART. The centers are inset so their 0.28 x 0.30 m
-           envelope remains inside the configured 0.32 x 0.31 m footprint. -->
-      <origin xyz="${-omni_contact_x_inset} 0 ${-omni_contact_y_inset}" rpy="0 0 0"/>
-      <geometry>
-        <sphere radius="${omni_contact_radius}"/>
-      </geometry>
-    </collision>
-    <xacro:default_inertial mass="0.5"/>
+    <xacro:unless value="$(arg use_cad_visual)">
+      <visual>
+        <geometry>
+          <cylinder length="${length_wheel}" radius="${radius_wheel}"/>
+        </geometry>
+        <material name="black"><color rgba="0.03 0.03 0.03 1"/></material>
+      </visual>
+    </xacro:unless>
+    <collision>
+      <geometry>
+        <sphere radius="${omni_contact_radius}"/>
+      </geometry>
+    </collision>
+    <xacro:sphere_inertial mass="${wheel_mass}" radius="${omni_contact_radius}" />
   </link>
   <link name="wheel_2">
-    <visual>
-      <geometry>
-        <cylinder length="${length_wheel}" radius="${radius_wheel}"/>
-      </geometry>
-      <origin rpy="0 0 0" xyz="0 0 0"/>
-      <material name="black"/>
-    </visual>
-    <collision>
-      <origin xyz="${omni_contact_x_inset} 0 ${-omni_contact_y_inset}" rpy="0 0 0"/>
-      <geometry>
-        <sphere radius="${omni_contact_radius}"/>
-      </geometry>
-    </collision>
-    <xacro:default_inertial mass="0.5"/>
+    <xacro:unless value="$(arg use_cad_visual)">
+      <visual><geometry><cylinder length="${length_wheel}" radius="${radius_wheel}"/></geometry><material name="black"/></visual>
+    </xacro:unless>
+    <collision>
+      <geometry>
+        <sphere radius="${omni_contact_radius}"/>
+      </geometry>
+    </collision>
+    <xacro:sphere_inertial mass="${wheel_mass}" radius="${omni_contact_radius}" />
   </link>
   <link name="wheel_3">
-    <visual>
-      <geometry>
-        <cylinder length="${length_wheel}" radius="${radius_wheel}"/>
-      </geometry>
-      <origin rpy="0 0 0" xyz="0 0 0"/>
-      <material name="black"/>
-    </visual>
-    <collision>
-      <origin xyz="${-omni_contact_x_inset} 0 ${omni_contact_y_inset}" rpy="0 0 0"/>
-      <geometry>
-        <sphere radius="${omni_contact_radius}"/>
-      </geometry>
-    </collision>
-    <xacro:default_inertial mass="0.5"/>
+    <xacro:unless value="$(arg use_cad_visual)">
+      <visual><geometry><cylinder length="${length_wheel}" radius="${radius_wheel}"/></geometry><material name="black"/></visual>
+    </xacro:unless>
+    <collision>
+      <geometry>
+        <sphere radius="${omni_contact_radius}"/>
+      </geometry>
+    </collision>
+    <xacro:sphere_inertial mass="${wheel_mass}" radius="${omni_contact_radius}" />
   </link>
   <link name="wheel_4">
-    <visual>
-      <geometry>
-        <cylinder length="${length_wheel}" radius="${radius_wheel}"/>
-      </geometry>
-      <origin rpy="0 0 0" xyz="0 0 0" />
-      <material name="black"/>
-    </visual>
-    <collision>
-      <origin xyz="${omni_contact_x_inset} 0 ${omni_contact_y_inset}" rpy="0 0 0"/>
-      <geometry>
-        <sphere radius="${omni_contact_radius}"/>
-      </geometry>
-    </collision>
-    <xacro:default_inertial mass="0.5"/>
+    <xacro:unless value="$(arg use_cad_visual)">
+      <visual><geometry><cylinder length="${length_wheel}" radius="${radius_wheel}"/></geometry><material name="black"/></visual>
+    </xacro:unless>
+    <collision>
+      <geometry>
+        <sphere radius="${omni_contact_radius}"/>
+      </geometry>
+    </collision>
+    <xacro:sphere_inertial mass="${wheel_mass}" radius="${omni_contact_radius}" />
   </link>
   <joint name="base_to_wheel1" type="fixed">
     <parent link="base_link"/>
     <child link="wheel_1"/>
-    <origin rpy="${-PI/2} 0 0" xyz="0.1 0.13 0"/>
+    <origin rpy="0 ${PI/2} ${-PI/4}" xyz="${wheel_center_offset} ${-wheel_center_offset} 0"/>
   </joint>
   <joint name="base_to_wheel2" type="fixed">
     <parent link="base_link"/>
     <child link="wheel_2"/>
-    <origin rpy="${-PI/2} 0 0" xyz="-0.1 0.13 0"/>
+    <origin rpy="0 ${PI/2} ${-PI/4}" xyz="${-wheel_center_offset} ${wheel_center_offset} 0"/>
   </joint>
   <joint name="base_to_wheel3" type="fixed">
     <parent link="base_link"/>
     <child link="wheel_3"/>
-    <origin rpy="${-PI/2} 0 0" xyz="0.1 -0.13 0"/>
+    <origin rpy="0 ${PI/2} ${PI/4}" xyz="${-wheel_center_offset} ${-wheel_center_offset} 0"/>
   </joint>
   <joint name="base_to_wheel4" type="fixed">
     <parent link="base_link"/>
     <child link="wheel_4"/>
-    <origin rpy="${-PI/2} 0 0" xyz="-0.1 -0.13 0"/>
+    <origin rpy="0 ${PI/2} ${PI/4}" xyz="${wheel_center_offset} ${wheel_center_offset} 0"/>
   </joint>
   <!-- IMU joint -->
@@ -149,16 +189,13 @@
       <origin xyz="0 0 0" rpy="0 0 0"/>
       <geometry>
-        <box size="0.05 0.05 0.05"/>
-      </geometry>
-    </collision>
-    <visual>
-      <origin xyz="0 0 0" rpy="0 0 0"/>
-      <geometry>
-        <box size="0.05 0.05 0.05"/>
-      </geometry>
-      <material name="green">
-        <color rgba="0 1 0 1"/>
-      </material>
-    </visual>
+        <box size="0.076 0.072 0.066"/>
+      </geometry>
+    </collision>
+    <xacro:unless value="$(arg use_cad_visual)">
+      <visual>
+        <geometry><box size="0.076 0.072 0.066"/></geometry>
+        <material name="green"><color rgba="0 1 0 1"/></material>
+      </visual>
+    </xacro:unless>
     <inertial>
       <mass value="1e-2" />
@@ -168,26 +205,37 @@
   </link>
   <!-- Gazebo插件设置相关 -->
-  <gazebo reference="base_link">
-    <material>Gazebo/Orange</material>
-  </gazebo>
+  <xacro:unless value="$(arg use_cad_visual)">
+    <gazebo reference="base_link"><material>Gazebo/Orange</material></gazebo>
+  </xacro:unless>
+  <!-- Bullet Featherstone shares one friction setting across a link's
+       compound collider. Keep the wheels separate so fixed-joint lumping
+       cannot replace their omni friction with the chassis default. -->
+  <gazebo reference="base_to_wheel1"><preserveFixedJoint>true</preserveFixedJoint></gazebo>
+  <gazebo reference="base_to_wheel2"><preserveFixedJoint>true</preserveFixedJoint></gazebo>
+  <gazebo reference="base_to_wheel3"><preserveFixedJoint>true</preserveFixedJoint></gazebo>
+  <gazebo reference="base_to_wheel4"><preserveFixedJoint>true</preserveFixedJoint></gazebo>
   <gazebo reference="wheel_1">
     <material>Gazebo/Red</material>
-    <mu1>0.05</mu1>
-    <mu2>0.05</mu2>
+    <mu1>${omni_friction}</mu1>
+    <mu2>${omni_friction}</mu2>
+    <xacro:bullet_omni_friction/>
   </gazebo>
   <gazebo reference="wheel_2">
     <material>Gazebo/Black</material>
-    <mu1>0.05</mu1>
-    <mu2>0.05</mu2>
+    <mu1>${omni_friction}</mu1>
+    <mu2>${omni_friction}</mu2>
+    <xacro:bullet_omni_friction/>
   </gazebo>
   <gazebo reference="wheel_3">
     <material>Gazebo/Red</material>
-    <mu1>0.05</mu1>
-    <mu2>0.05</mu2>
+    <mu1>${omni_friction}</mu1>
+    <mu2>${omni_friction}</mu2>
+    <xacro:bullet_omni_friction/>
   </gazebo>
   <gazebo reference="wheel_4">
     <material>Gazebo/Black</material>
-    <mu1>0.05</mu1>
-    <mu2>0.05</mu2>
+    <mu1>${omni_friction}</mu1>
+    <mu2>${omni_friction}</mu2>
+    <xacro:bullet_omni_friction/>
   </gazebo>
   <gazebo reference="imu_link">
@@ -240,5 +288,6 @@
   <!-- Livox-Mid360  -->
   <xacro:include filename="$(find rm_27_stimulation)/urdf/mid360.xacro" />
-  <xacro:mid360 name="left_mid360" parent="base_link" topic="/livox/lidar">
+  <xacro:mid360 name="left_mid360" parent="base_link" topic="/livox/lidar"
+                  hide_visual="$(arg use_cad_visual)">
     <origin xyz="$(arg xyz)" rpy="$(arg rpy)" />
   </xacro:mid360>

Commit message: [update]解决了过洞误识别，以及小车与静态障碍物重叠停止移动的问题

File: src/rm_27_stimulation/urdf/mid360.xacro (robot description, xacro)
@@ -53,9 +53,8 @@
             </horizontal>
             <vertical>
-              <!-- 96 elevation rings keep the nearest ground-return spacing
-                   below one 5 cm ROG cell while avoiding a 115200-ray Gazebo
-                   bottleneck. Horizontal samples remain 360 for doorway
-                   width resolution; total rays are 34560. -->
-              <samples>96</samples>
+              <!-- More than 128 rings selects a 256 px Ogre2 depth cubemap.
+                   The 128 px cubemap biases a 250 mm opening below the
+                   240 mm chassis height. Keep the localizer layout in sync. -->
+              <samples>192</samples>
               <resolution>1</resolution>
               <min_angle>${-7.22/180*M_PI}</min_angle>

File: src/rm_27_stimulation/urdf/simulation_waking_robot.xacro (robot description, xacro)
@@ -7,4 +7,8 @@
   <xacro:property name="omni_contact_radius" value="${radius_wheel}" />
   <xacro:property name="wheel_center_offset" value="0.218" />
+  <xacro:property name="folded_vehicle_height" value="0.240" />
+  <xacro:property name="folded_top_z" value="${folded_vehicle_height - radius_wheel}" />
+  <xacro:property name="cad_body_z_scale" value="${folded_top_z / 0.16638150811195374}" />
+  <xacro:property name="cad_sensor_z_scale" value="${(folded_top_z - 0.130) / (0.168313 - 0.130)}" />
   <xacro:property name="omni_friction" value="0.05" />
   <xacro:property name="body_mass" value="8.2" />
@@ -32,10 +36,11 @@
     </inertial>
   </xacro:macro>
-  <xacro:macro name="cad_visual" params="mesh material">
+  <xacro:macro name="cad_visual" params="mesh material z_scale:=1.0 z_origin:=0.0">
     <visual>
       <geometry>
         <mesh filename="package://rm_27_stimulation/meshes/rm27_sentry_visual/${mesh}.stl"
-              scale="$(arg cad_visual_scale) $(arg cad_visual_scale) $(arg cad_visual_scale)" />
-      </geometry>
+              scale="$(arg cad_visual_scale) $(arg cad_visual_scale) ${float('$(arg cad_visual_scale)') * z_scale}" />
+      </geometry>
+      <origin xyz="0 0 ${float('$(arg cad_visual_scale)') * z_origin}" />
       <material name="${material}" />
     </visual>
@@ -61,8 +66,9 @@
   <link name="base_link">
     <xacro:if value="$(arg use_cad_visual)">
-      <xacro:cad_visual mesh="body" material="cad_body" />
+      <xacro:cad_visual mesh="body" material="cad_body" z_scale="${cad_body_z_scale}" />
       <xacro:cad_visual mesh="wheels" material="cad_wheels" />
-      <xacro:cad_visual mesh="armor" material="cad_armor" />
-      <xacro:cad_visual mesh="sensors" material="cad_sensors" />
+      <xacro:cad_visual mesh="armor" material="cad_armor" z_scale="${cad_body_z_scale}" />
+      <xacro:cad_visual mesh="sensors" material="cad_sensors" z_scale="${cad_sensor_z_scale}"
+                        z_origin="${0.130 * (1.0 - cad_sensor_z_scale)}" />
     </xacro:if>
     <xacro:unless value="$(arg use_cad_visual)">
@@ -87,11 +93,12 @@
     <collision>
       <geometry>
-        <box size="0.48 0.48 0.08" />
-      </geometry>
-      <origin rpy="0 0 0" xyz="0 0 0.14" />
+        <!-- Keep the folded collision top 240 mm above the wheel contact plane. -->
+        <box size="0.362 0.354 0.040" />
+      </geometry>
+      <origin rpy="0 0 0" xyz="-0.043 -0.016 ${folded_top_z - 0.020}" />
     </collision>
     <!-- STL has no material density. Preserve the validated 10.2 kg total
          mass, but derive the inertia from the CAD body envelope. -->
-    <xacro:box_inertial mass="${body_mass}" x="0.54" y="0.54" z="0.20"
+    <xacro:box_inertial mass="${body_mass}" x="0.54" y="0.54" z="${0.20 * cad_body_z_scale}"
                          ox="0.0" oy="0.0" oz="0.066" />
   </link>
@@ -189,10 +196,10 @@
       <origin xyz="0 0 0" rpy="0 0 0"/>
       <geometry>
-        <box size="0.076 0.072 0.066"/>
+        <box size="0.076 0.048 0.040"/>
       </geometry>
     </collision>
     <xacro:unless value="$(arg use_cad_visual)">
       <visual>
-        <geometry><box size="0.076 0.072 0.066"/></geometry>
+        <geometry><box size="0.076 0.048 0.040"/></geometry>
         <material name="green"><color rgba="0 1 0 1"/></material>
       </visual>
@@ -269,6 +276,5 @@
       <max_yaw_torque>8.0</max_yaw_torque>
     </plugin>
-    <plugin filename="gz-sim-odometry-publisher-system" name="gz::sim::systems::OdometryPublisher">
-      <dimensions>3</dimensions>
+    <plugin filename="librm27_ground_truth_odometry_system.so" name="rm_27_stimulation::GroundTruthOdometrySystem">
       <odom_publish_frequency>50</odom_publish_frequency>
       <odom_topic>/ground_truth/odometry</odom_topic>
