Commit message: [update]解决了gazebo渲染以及其他问题，修改仿真小车模型

File: src/rm_27_stimulation/urdf/simulation_waking_robot.xacro (robot description, xacro)
@@ -12,21 +12,21 @@
   </xacro:macro>
   <!-- Logical Mid360 frame relative to base_link; physical roll is compensated before this frame. -->
-  <xacro:arg name="xyz" default="0.0 0.18 0.28" />
+  <xacro:arg name="xyz" default="0.0 0.18 0.14" />
   <xacro:arg name="rpy" default="0 0 0" />
   <link name="base_link">
     <visual>
       <geometry>
-        <box size="0.2 .3 .1"/>
-      </geometry>
-      <origin rpy="0 0 ${PI/2}" xyz="0 0 0.05"/>
-      <material name="white">
-        <color rgba="1 1 1 1"/>
+        <box size="0.2 .3 .14"/>
+      </geometry>
+      <origin rpy="0 0 ${PI/2}" xyz="0 0 0.07"/>
+      <material name="orange">
+        <color rgba="0.95 0.28 0.04 1"/>
       </material>
     </visual>
     <collision>
       <geometry>
-        <box size="0.2 .3 0.1"/>
-      </geometry>
-      <origin rpy="0 0 ${PI/2}" xyz="0 0 0.05"/>
+        <box size="0.2 .3 0.14"/>
+      </geometry>
+      <origin rpy="0 0 ${PI/2}" xyz="0 0 0.07"/>
     </collision>
     <xacro:default_inertial mass="8.2"/>
@@ -59,6 +59,4 @@
       </geometry>
     </collision>
-    <mu1>0.5</mu1>
-    <mu2>0.5</mu2>
     <xacro:default_inertial mass="0.5"/>
   </link>
@@ -76,6 +74,4 @@
       </geometry>
     </collision>
-    <mu1>0.5</mu1>
-    <mu2>0.5</mu2>
     <xacro:default_inertial mass="0.5"/>
   </link>
@@ -93,6 +89,4 @@
       </geometry>
     </collision>
-    <mu1>0.5</mu1>
-    <mu2>0.5</mu2>
     <xacro:default_inertial mass="0.5"/>
   </link>
@@ -110,6 +104,4 @@
       </geometry>
     </collision>
-    <mu1>0.5</mu1>
-    <mu2>0.5</mu2>
     <xacro:default_inertial mass="0.5"/>
   </link>
@@ -170,13 +162,21 @@
   <gazebo reference="wheel_1">
     <material>Gazebo/Red</material>
+    <mu1>0.05</mu1>
+    <mu2>0.05</mu2>
   </gazebo>
   <gazebo reference="wheel_2">
     <material>Gazebo/Black</material>
+    <mu1>0.05</mu1>
+    <mu2>0.05</mu2>
   </gazebo>
   <gazebo reference="wheel_3">
     <material>Gazebo/Red</material>
+    <mu1>0.05</mu1>
+    <mu2>0.05</mu2>
   </gazebo>
   <gazebo reference="wheel_4">
     <material>Gazebo/Black</material>
+    <mu1>0.05</mu1>
+    <mu2>0.05</mu2>
   </gazebo>
   <gazebo reference="imu_link">
@@ -194,4 +194,15 @@
       <max_linear_velocity>3.0</max_linear_velocity>
       <max_angular_velocity>6.0</max_angular_velocity>
+      <linear_velocity_gain>80.0</linear_velocity_gain>
+      <angular_velocity_gain>4.0</angular_velocity_gain>
+      <max_planar_force>120.0</max_planar_force>
+      <max_yaw_torque>8.0</max_yaw_torque>
+    </plugin>
+    <plugin filename="gz-sim-odometry-publisher-system" name="gz::sim::systems::OdometryPublisher">
+      <dimensions>3</dimensions>
+      <odom_publish_frequency>50</odom_publish_frequency>
+      <odom_topic>/ground_truth/odometry</odom_topic>
+      <odom_frame>world</odom_frame>
+      <robot_base_frame>base_footprint</robot_base_frame>
     </plugin>
   </gazebo>

Commit message: [update]新增仿真立头倒头和云台旋转功能，优化rog_map障碍物清除逻辑，调整实车仿真参数

File: src/rm_27_stimulation/urdf/simulation_waking_robot.xacro (robot description, xacro)
@@ -12,5 +12,5 @@
   <xacro:property name="cad_sensor_z_scale" value="${(folded_top_z - 0.130) / (0.168313 - 0.130)}" />
   <xacro:property name="omni_friction" value="0.05" />
-  <xacro:property name="body_mass" value="8.2" />
+  <xacro:property name="body_mass" value="5.0" />
   <xacro:property name="wheel_mass" value="0.5" />
   <xacro:property name="PI" value="3.1415926"/>
@@ -66,9 +66,7 @@
   <link name="base_link">
     <xacro:if value="$(arg use_cad_visual)">
-      <xacro:cad_visual mesh="body" material="cad_body" z_scale="${cad_body_z_scale}" />
+      <xacro:cad_visual mesh="chassis_body" material="cad_body" />
       <xacro:cad_visual mesh="wheels" material="cad_wheels" />
-      <xacro:cad_visual mesh="armor" material="cad_armor" z_scale="${cad_body_z_scale}" />
-      <xacro:cad_visual mesh="sensors" material="cad_sensors" z_scale="${cad_sensor_z_scale}"
-                        z_origin="${0.130 * (1.0 - cad_sensor_z_scale)}" />
+      <xacro:cad_visual mesh="chassis_armor" material="cad_armor" />
     </xacro:if>
     <xacro:unless value="$(arg use_cad_visual)">
@@ -91,11 +89,4 @@
       <origin rpy="0 0 0" xyz="0 0 0.06" />
     </collision>
-    <collision>
-      <geometry>
-        <!-- Keep the folded collision top 240 mm above the wheel contact plane. -->
-        <box size="0.362 0.354 0.040" />
-      </geometry>
-      <origin rpy="0 0 0" xyz="-0.043 -0.016 ${folded_top_z - 0.020}" />
-    </collision>
     <!-- STL has no material density. Preserve the validated 10.2 kg total
          mass, but derive the inertia from the CAD body envelope. -->
@@ -109,9 +100,41 @@
     <origin xyz="0 0 0" rpy="0 0 0"/>
   </joint>
-  <link name="gimbal_yaw"/>
-  <joint name="gimbal_yaw_joint" type="fixed">
+  <link name="gimbal_yaw">
+    <xacro:if value="$(arg use_cad_visual)">
+      <xacro:cad_visual mesh="yaw_body" material="cad_body" />
+      <xacro:cad_visual mesh="yaw_sensors" material="cad_sensors" />
+    </xacro:if>
+    <collision>
+      <origin xyz="-0.073114 -0.031 0.082082"/>
+      <geometry><box size="0.298 0.378 0.155837"/></geometry>
+    </collision>
+    <xacro:box_inertial mass="2.4" x="0.298" y="0.378" z="0.155837"
+                       ox="-0.073114" oy="-0.031" oz="0.082082"/>
+  </link>
+  <joint name="gimbal_yaw_joint" type="continuous">
     <parent link="base_link"/>
     <child link="gimbal_yaw"/>
-    <origin xyz="0 0 0.12" rpy="0 0 0"/>
+    <origin xyz="0 0 0" rpy="0 0 0"/>
+    <axis xyz="0 0 1"/>
+    <limit effort="5.0" velocity="1.2"/>
+    <dynamics damping="0.05" friction="0.0"/>
+  </joint>
+  <link name="gimbal_roll">
+    <xacro:if value="$(arg use_cad_visual)">
+      <xacro:cad_visual mesh="roll_body" material="cad_body" />
+    </xacro:if>
+    <collision>
+      <origin xyz="0.151083 -0.064732 -0.000066"/>
+      <geometry><box size="0.246119 0.297858 0.125430"/></geometry>
+    </collision>
+    <xacro:box_inertial mass="0.8" x="0.246119" y="0.297858" z="0.125430"
+                       ox="0.151083" oy="-0.064732" oz="-0.000066"/>
+  </link>
+  <joint name="gimbal_roll_joint" type="revolute">
+    <parent link="gimbal_yaw"/><child link="gimbal_roll"/>
+    <origin xyz="0.005862518 0.015803345 0.087848857"/>
+    <axis xyz="-1 0 0"/>
+    <limit lower="0.0" upper="${PI/2}" effort="5.0" velocity="1.0"/>
+    <dynamics damping="0.05" friction="0.0"/>
   </joint>
   <link name="wheel_1">
@@ -188,5 +211,5 @@
     <axis xyz="0 1 0" />
     <origin xyz="$(arg xyz)" rpy="$(arg rpy)"/>
-    <parent link="base_link"/>
+    <parent link="gimbal_yaw"/>
     <child link="imu_link"/>
   </joint>
@@ -254,4 +277,18 @@
   <!-- Drive controller plugin -->
   <gazebo>
+    <plugin filename="gz-sim-joint-position-controller-system" name="gz::sim::systems::JointPositionController">
+      <joint_name>gimbal_yaw_joint</joint_name><topic>/sim/gimbal/yaw_position</topic>
+      <p_gain>40</p_gain><i_gain>5</i_gain><d_gain>2</d_gain>
+      <i_max>2</i_max><i_min>-2</i_min><cmd_max>5</cmd_max><cmd_min>-5</cmd_min>
+    </plugin>
+    <plugin filename="gz-sim-joint-position-controller-system" name="gz::sim::systems::JointPositionController">
+      <joint_name>gimbal_roll_joint</joint_name><topic>/sim/gimbal/roll_position</topic>
+      <p_gain>40</p_gain><i_gain>5</i_gain><d_gain>2</d_gain>
+      <i_max>2</i_max><i_min>-2</i_min><cmd_max>5</cmd_max><cmd_min>-5</cmd_min>
+    </plugin>
+    <plugin filename="gz-sim-joint-state-publisher-system" name="gz::sim::systems::JointStatePublisher">
+      <joint_name>gimbal_yaw_joint</joint_name><joint_name>gimbal_roll_joint</joint_name>
+      <topic>/sim/gimbal/joint_states</topic>
+    </plugin>
     <plugin name="rm_27_stimulation::CmdVelPoseControlSystem" filename="librm27_cmd_vel_pose_control_system.so">
       <topic>/cmd_vel</topic>
@@ -294,5 +331,5 @@
   <!-- Livox-Mid360  -->
   <xacro:include filename="$(find rm_27_stimulation)/urdf/mid360.xacro" />
-  <xacro:mid360 name="left_mid360" parent="base_link" topic="/livox/lidar"
+  <xacro:mid360 name="left_mid360" parent="gimbal_yaw" topic="/livox/lidar"
                   hide_visual="$(arg use_cad_visual)">
     <origin xyz="$(arg xyz)" rpy="$(arg rpy)" />

File: src/sentry_robot_description/urdf/sentry_robot.urdf.xacro (robot description, xacro)
@@ -12,5 +12,5 @@
       <origin xyz="0 0 0.05" rpy="0 0 0"/>
       <geometry>
-        <box size="0.30 0.20 0.10"/>
+        <box size="0.50 0.50 0.10"/>
       </geometry>
       <material name="body_gray">
@@ -18,4 +18,10 @@
       </material>
     </visual>
+    <collision>
+      <origin xyz="0 0 0.05" rpy="0 0 0"/>
+      <geometry>
+        <box size="0.50 0.50 0.10"/>
+      </geometry>
+    </collision>
   </link>
   <joint name="base_footprint_joint" type="fixed">
